File: dsp.brd (EAGLE design)
At the start: 190 x 113 mm, 131 parts, among them IC1 OPA2134P, IC2 OPA2134P, IC3 OPA2134P, U1 STM32F405RGT6, U2 CODECODER-WM8731SEDS/V(SSOP28), U4 LM2575HVS-3.3/NOPB, X1 ABLS-8.000MHZ-B4-T

Commit message: sent it out to get made
Parts:
- removed LED2: TLLG4400, dan:LED3MM
- added LED1: (no value), dan:LED5MM
- POWER: value TLLG4400 -> (none); device dan:LED3MM -> dan:LED5MM
- moved R8 3.21 mm to (7.62, 19.1)
- moved C21 1.61 mm to (74.7, 27.4)
- moved R1 1.02 mm to (35.3, 100.8)
- moved C2 1.02 mm to (21.1, 82.8)
- moved C18 0.76 mm to (72.4, 62.2)
- moved U$2 0.51 mm to (43.2, 103.6)
Connections:
- removed net HPVDD: U2.8
- new net N$60: IC3.6, IC3.7
- net 3.3V: now also U2.8
- net GND: now also IC3.5, U2.11
- net N$10: now also LED1.K; no longer LED2.K
- net N$9: now also LED1.A; no longer LED2.A
Routing:
- net 3.3V: track 564.5 -> 581.5 mm
- net N$60: track 0.00 -> 2.54 mm
- net N$9: track 33.7 -> 35.8 mm
- net FBR: track 84.5 -> 83.2 mm
- net N$6: track 4.37 -> 5.49 mm
- net ROUT: track 20.3 -> 21.3 mm
- net NRESET: track 65.5 -> 64.6 mm
- net N$17: track 28.7 -> 27.9 mm
- net LIN: track 22.1 -> 22.9 mm
Other:
- outline, holes or cut-outs redrawn
